File: Schematic/bms/bms/BMS_BQ76920.kicad_sch (KiCad schematic)
At the start: 33 parts, among them J2 5267-05A-X, J3 5267-05A-X, Q1 CSD17581Q5A, Q3 PMOS, U1 BQ76920PW

Commit message: Update
Other:
- note added: "MOSFET은 도통되면 Source, Drain 어느 방향으로도 전류의 흐름이 가능 Q1/CHG ON 충전/방전 둘 다 허용 OFF 충전 차단 (과충전) 과방전 조건: UV(셀 저전압)/OCD(방전 과전류)/SCD(단락 보호) 드론의 방전을 차단하면 위험하다 판단해서 뺐음"
- note removed: "MOSFET은 도통되면 Source, Drain 어느 방향으로도 전류의 흐름이 가능 Q1/DSG Q2/CHG ON ON 충전/방전 둘 다 허용 ON OFF 충전 차단 (과충전) OFF ON 방전 차단 (과방전/과전류/단락) OFF OFF 양방향 차단 (완전 보호) 과방전 조건: UV(셀 저전압)/OCD(방전 과전류)/SCD(단락 보호) 드론의 방전을 차단하면 위험하다 판단해서 뺐음"
Changed lines of the file:
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@@
 		)
 	)
-	(text "MOSFET은 도통되면 Source, Drain 어느 방향으로도 전류의 흐름이 가능\n\nQ1/DSG		Q2/CHG\nON  			ON 		충전/방전 둘 다 허용 \nON				OFF 		충전 차단 (과충전)\nOFF			ON			방전 차단 (과방전/과전류/단락)\nOFF			OFF		양방향 차단 (완전 보호)\n\n과방전 조건: UV(셀 저전압)/OCD(방전 과전류)/SCD(단락 보호)\n\n드론의 방전을 차단하면 위험하다 판단해서 뺐음"
+	(text "MOSFET은 도통되면 Source, Drain 어느 방향으로도 전류의 흐름이 가능\n\nQ1/CHG\nON 			충전/방전 둘 다 허용 \nOFF 			충전 차단 (과충전)\n\n과방전 조건: UV(셀 저전압)/OCD(방전 과전류)/SCD(단락 보호)\n\n드론의 방전을 차단하면 위험하다 판단해서 뺐음"
 		(exclude_from_sim no)
 		(at 137.16 148.59 0)

Commit message: Update
Connections:
- net VBAT: now also J2.5, R8.1
Other:
- moved on the sheet: C10, C11, C7, C8, C9, J2, R10, R11, R12, R8, R9

Commit message: Update
Parts:
- removed Q1: CSD17581Q5A, MOSFET_IC:MOSFET_CSD19531Q5A, symbol Simulation_SPICE:NMOS
- added Q2: CSD17581Q3A, Package_SON:VSON-8_3.3x3.3mm_P0.65mm_NexFET, symbol Transistor_FET:CSD17581Q3A
- C14: renamed from C11; footprint (none) -> Capacitor_SMD:C_0805_2012Metric_Pad1.18x1.45mm_HandSolder
- C15: renamed from C7; footprint (none) -> Capacitor_SMD:C_0805_2012Metric_Pad1.18x1.45mm_HandSolder
- C16: renamed from C8; footprint (none) -> Capacitor_SMD:C_0805_2012Metric_Pad1.18x1.45mm_HandSolder
- C17: renamed from C9; footprint (none) -> Capacitor_SMD:C_0805_2012Metric_Pad1.18x1.45mm_HandSolder
- C18: renamed from C10; footprint (none) -> Capacitor_SMD:C_0805_2012Metric_Pad1.18x1.45mm_HandSolder
- C19: renamed from C4; footprint (none) -> Capacitor_SMD:C_0805_2012Metric_Pad1.18x1.45mm_HandSolder
- C20: renamed from C1; footprint (none) -> Capacitor_SMD:C_0805_2012Metric_Pad1.18x1.45mm_HandSolder
- C21: renamed from C3; footprint (none) -> Capacitor_SMD:C_0805_2012Metric_Pad1.18x1.45mm_HandSolder
- C22: renamed from C2; footprint (none) -> Capacitor_SMD:C_0805_2012Metric_Pad1.18x1.45mm_HandSolder
- D5: renamed from D1; footprint (none) -> Diode_SMD:D_SOD-123
- D6: renamed from D2; footprint (none) -> Diode_SMD:D_SOD-123
- Q1: renamed from Q3; footprint (none) -> Package_TO_SOT_SMD:SOT-323_SC-70_Handsoldering
- R14: renamed from R8; footprint (none) -> Resistor_SMD:R_0805_2012Metric_Pad1.20x1.40mm_HandSolder
- R15: renamed from R11; footprint (none) -> Resistor_SMD:R_0805_2012Metric_Pad1.20x1.40mm_HandSolder
- R16: renamed from R9; footprint (none) -> Resistor_SMD:R_0805_2012Metric_Pad1.20x1.40mm_HandSolder
- R17: renamed from R12; footprint (none) -> Resistor_SMD:R_0805_2012Metric_Pad1.20x1.40mm_HandSolder
- R18: renamed from R10; footprint (none) -> Resistor_SMD:R_0805_2012Metric_Pad1.20x1.40mm_HandSolder
- R19: renamed from R1; footprint (none) -> Resistor_SMD:R_0805_2012Metric_Pad1.20x1.40mm_HandSolder
- R20: renamed from R2; footprint (none) -> Resistor_SMD:R_Shunt_Vishay_WSR2_WSR3
- R21: renamed from R3; footprint (none) -> Resistor_SMD:R_0805_2012Metric_Pad1.20x1.40mm_HandSolder
- R22: renamed from R14; footprint (none) -> Resistor_SMD:R_0805_2012Metric_Pad1.20x1.40mm_HandSolder
- R23: renamed from R13; footprint (none) -> Resistor_SMD:R_0805_2012Metric_Pad1.20x1.40mm_HandSolder
- R24: renamed from R19; footprint (none) -> Resistor_SMD:R_0805_2012Metric_Pad1.20x1.40mm_HandSolder
- R25: renamed from R16; footprint (none) -> Resistor_SMD:R_0805_2012Metric_Pad1.20x1.40mm_HandSolder
- R26: renamed from R15; footprint (none) -> Resistor_SMD:R_0805_2012Metric_Pad1.20x1.40mm_HandSolder
- R27: renamed from R5; footprint (none) -> Resistor_SMD:R_0805_2012Metric_Pad1.20x1.40mm_HandSolder
- R28: renamed from R7; footprint (none) -> Resistor_SMD:R_0805_2012Metric_Pad1.20x1.40mm_HandSolder
- R29: renamed from R6; footprint (none) -> Resistor_SMD:R_0805_2012Metric_Pad1.20x1.40mm_HandSolder
- TH1: footprint (none) -> Resistor_SMD:R_0805_2012Metric_Pad1.20x1.40mm_HandSolder
- renumbered J2 to J21, J3 to J22, U1 to U3
Connections:
- net PACK-: now also Q2.1 (S), Q2.2 (S), Q2.3 (S)
- net at R20.1, R21.1: now also Q2.5 (D)
- net at D6.1 (K), R25.2, R26.2: now also Q2.4 (G)
- net +3V3 renamed REGOUT
