File: Schematic/bms/bms/bms.kicad_sch (KiCad schematic)
At the start: 40 parts, among them J1 XT60-M, J10 M4 Vcc, J11 M4 GND, J12 5V, J13 GND, J14 3.3V, J15 GND, J16 5V, J17 3.3V, J18 3.3V, J19 3.3V, J22 Battery Charge, J4 M1 Vcc, J5 M1 GND, J6 M2 Vcc, J7 M2 GND, J8 M3 Vcc, J9 M3 GND, U2 LMR51450SDRRR, U3 TPS54302

Commit message: Update
Parts:
- added D4, D5: D_Schottky_Small, symbol Device:D_Schottky_Small
- added D6: LED_Green, symbol Device:LED_Small
- added R23: 2.2k, symbol Device:R_Small
- R22: value 1k -> 2.2k
Connections:
- net +3V3: now also R23.1
- net SGND: now also D3.1 (K), D6.1 (K)
- net VBAT: now also D4.1 (K), D5.1 (K)
- net at C12.1, U2.4 (BOOT): now also D5.2 (A)
- net at C17.2, L1.1, U3.2 (SW): now also D4.2 (A)
- net PG: no longer names the net of U2.5 (PG)
- net PG: no longer D3.1 (K)
- new net: D6.2 (A), R23.2
- no-connect marks 0 -> 1
Other:
- note added: "Buck 외부 회로 부품 선정"
- note added: "스위칭 주파수 선택 기준"
- moved on the sheet: C16, C17, C18, D3, J1, L1, R22, R24, R25, U3

Commit message: Update
Connections:
- net at C12.2, L2.1, U2.1 (SW)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: now also D5.2 (A)
- net at C12.1, U2.4 (BOOT): no longer D5.2 (A)
Other:
- moved on the sheet: L2
Changed lines of the file:
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@@
 		)
 	)
-	(text_box "1. 낮은 주파수 (200~400kHz)\n- 장점: 스위칭 손실이 적어 효율↑, 발열↓\n- 단점: 인덕터와 커패시터 값이 커져서 부품 크기↑\n\n2. 중간 주파수 (500 kHz, 기본값)\n- 장점: 효율과 크기 사이의 균형\n- TI 기본 권장값\n\n3. 높은 주파수 (800 kHz~1 MHz)\n- 장점: 인덕터·커패시터 값이 작아져서 PCB 크기↓\n- 단점: 스위칭 손실↑, 발열↑, 효율↓"
+	(text_box "1. 낮은 주파수 (200k~400kHz)\n- 장점: 스위칭 손실이 적어 효율↑, 발열↓\n- 단점: 인덕터와 커패시터 값이 커져서 부품 크기↑\n\n2. 중간 주파수 (500kHz, 기본값)\n- 장점: 효율과 크기 사이의 균형\n- TI 기본 권장값\n\n3. 높은 주파수 (800kHz~1MHz)\n- 장점: 인덕터·커패시터 값이 작아져서 PCB 크기↓\n- 단점: 스위칭 손실↑, 발열↑, 효율↓"
 		(exclude_from_sim no)
 		(at 205.74 21.59 0)
@@
 	)
 	(junction
+		(at 135.89 43.18)
+		(diameter 0)
+		(color 0 0 0 0)
+	)
+	(junction
 		(at 82.55 109.22)
 		(diameter 0)
@@
 	)
 	(junction
-		(at 129.54 38.1)
-		(diameter 0)
-		(color 0 0 0 0)
-	)
-	(junction
 		(at 147.32 43.18)
 		(diameter 0)
@@
 	(wire
 		(pts
+			(xy 129.54 43.18) (xy 135.89 43.18)
+		)
+		(stroke
+			(width 0)
+			(type default)
+		)
+	)
+	(wire
+		(pts
 			(xy 39.37 166.37) (xy 39.37 170.18)
 		)
@@
 	(wire
 		(pts
+			(xy 137.16 43.18) (xy 135.89 43.18)
+		)
+		(stroke
+			(width 0)
+			(type default)
+		)
+	)
+	(wire
+		(pts
 			(xy 214.63 62.23) (xy 214.63 67.31)
 		)
@@
 	(wire
 		(pts
-			(xy 129.54 43.18) (xy 135.89 43.18)
-		)
-		(stroke
-			(width 0)
-			(type default)
-		)
-	)
-	(wire
-		(pts
 			(xy 220.98 116.84) (xy 214.63 116.84)
 		)
@@
 	(wire
 		(pts
-			(xy 143.51 43.18) (xy 147.32 43.18)
+			(xy 144.78 43.18) (xy 147.32 43.18)
 		)
 		(stroke
@@
 	(wire
 		(pts
-			(xy 129.54 26.67) (xy 109.22 26.67)
+			(xy 135.89 26.67) (xy 109.22 26.67)
 		)
 		(stroke
@@
 	(wire
 		(pts
-			(xy 129.54 38.1) (xy 129.54 26.67)
+			(xy 135.89 26.67) (xy 135.89 43.18)
 		)
 		(stroke
@@
 	(symbol
 		(lib_id "0_Basic_Components:L")
-		(at 139.7 43.18 90)
+		(at 140.97 43.18 90)
 		(unit 1)
 		(exclude_from_sim no)
@@
 		(fields_autoplaced yes)
 		(property "Reference" "L2"
-			(at 139.7 38.1 90)
+			(at 140.97 38.1 90)
 			(effects
 				(font
@@
 		)
 		(property "Value" "L"
-			(at 139.7 40.64 90)
+			(at 140.97 40.64 90)
 			(effects
 				(font
@@
 		)
 		(property "Footprint" ""
-			(at 139.7 43.18 0)
+			(at 140.97 43.18 0)
 			(effects
 				(font
@@
 		)
 		(property "Datasheet" "~"
-			(at 139.7 43.18 0)
+			(at 140.97 43.18 0)
 			(effects
 				(font
@@
 		)
 		(property "Description" "Inductor"
-			(at 139.7 43.18 0)
+			(at 140.97 43.18 0)
 			(effects
 				(font

Commit message: Update
Parts:
- removed C15: 33uF, symbol Device:C_Small
- removed C17: ~, symbol Device:C_Small
- removed J4: M1 Vcc, Connector_Wire:SolderWirePad_1x01_SMD_4x8mm, symbol Connector_Generic:Conn_01x01
- removed J6: M2 Vcc, Connector_Wire:SolderWirePad_1x01_SMD_4x8mm, symbol Connector_Generic:Conn_01x01
- removed J7: M2 GND, Connector_Wire:SolderWirePad_1x01_SMD_4x8mm, symbol Connector_Generic:Conn_01x01
- removed L1: L, symbol 0_Basic_Components:L
- removed R4: 0, symbol Device:R_Small
- removed U3: TPS54302, Package_TO_SOT_SMD:SOT-23-6, symbol Regulator_Switching:TPS54302
- added C1, C3: 10uF, Capacitor_SMD:C_0805_2012Metric_Pad1.18x1.45mm_HandSolder, symbol Device:C_Small
- added C10: 47uF, Capacitor_SMD:C_0805_2012Metric_Pad1.18x1.45mm_HandSolder, symbol Device:C_Small
- added C12: 33uF, Capacitor_SMD:C_0805_2012Metric_Pad1.18x1.45mm_HandSolder, symbol Device:C_Small
- added C13: 100uF, Capacitor_SMD:CP_Elec_6.3x5.9, symbol Device:C_Polarized_Small_US
- added C6: 0.1uF, Capacitor_SMD:C_0805_2012Metric_Pad1.18x1.45mm_HandSolder, symbol Device:C_Small
- added J10: 3.3V, Connector_Wire:SolderWirePad_1x01_SMD_2x4mm, symbol Connector_Generic:Conn_01x01
- added J12, J13, J14, J15: GND, Connector_Wire:SolderWirePad_1x01_SMD_2x4mm, symbol Connector_Generic:Conn_01x01
- added R2, R3, R6, R8: 0, Resistor_SMD:R_0805_2012Metric_Pad1.20x1.40mm_HandSolder, symbol Device:R_Small
- added R7: 100k, Resistor_SMD:R_0805_2012Metric_Pad1.20x1.40mm_HandSolder, symbol Device:R_Small
- added U2: TPSM53602RDA, Package_DFN_QFN:Texas_B3QFN-14-1EP_5x5.5mm_P0.65mm_ThermalVia, symbol Converter_DCDC:TPSM53602RDA
- C11: renamed from C14; footprint (none) -> Capacitor_SMD:C_0805_2012Metric_Pad1.18x1.45mm_HandSolder
- C2: renamed from C5; footprint (none) -> Capacitor_SMD:C_0805_2012Metric_Pad1.18x1.45mm_HandSolder
- C4: renamed from C6; value 1uF -> 0.1uF; footprint (none) -> Capacitor_SMD:C_0805_2012Metric_Pad1.18x1.45mm_HandSolder
- C5: renamed from C16; value ~ -> 10uF; footprint (none) -> Capacitor_SMD:C_0805_2012Metric_Pad1.18x1.45mm_HandSolder
- C7: renamed from C12; value 1uF -> 0.1uF; footprint (none) -> Capacitor_SMD:C_0805_2012Metric_Pad1.18x1.45mm_HandSolder
- C8: renamed from C18; value ~ -> 47uF; footprint (none) -> Capacitor_SMD:C_0805_2012Metric_Pad1.18x1.45mm_HandSolder
- C9: renamed from C13; footprint (none) -> Capacitor_SMD:C_0805_2012Metric_Pad1.18x1.45mm_HandSolder
- D1: renamed from D3; footprint (none) -> LED_SMD:LED_1206_3216Metric_Pad1.42x1.75mm_HandSolder
- D2: renamed from D6; footprint (none) -> LED_SMD:LED_1206_3216Metric_Pad1.42x1.75mm_HandSolder
- D3: renamed from D5; value D_Schottky_Small -> SS34; footprint (none) -> Diode_SMD:D_SMA_Handsoldering
- D4: value D_Schottky_Small -> SS34; footprint (none) -> Diode_SMD:D_SMA_Handsoldering
- J1: footprint Connector_AMASS:AMASS_XT60-M_1x02_P7.20mm_Vertical -> XT60-M:XT60-M_1x02_P7.20mm_Vertical
- J5: value M1 GND -> GND; footprint Connector_Wire:SolderWirePad_1x01_SMD_4x8mm -> Connector_Wire:SolderWirePad_1x01_SMD_2x4mm
- L1: renamed from L2; value L -> 4.7uH; footprint (none) -> Inductor_SMD:L_7.3x7.3_H3.5
- R1: renamed from R22; footprint (none) -> Resistor_SMD:R_0805_2012Metric_Pad1.20x1.40mm_HandSolder
- R10: renamed from R25; value ~ -> 4.32k; footprint (none) -> Resistor_SMD:R_0805_2012Metric_Pad1.20x1.40mm_HandSolder
- R11: renamed from R20; footprint (none) -> Resistor_SMD:R_0805_2012Metric_Pad1.20x1.40mm_HandSolder
- R12: renamed from R18; value 19.1k -> 18.6k; footprint (none) -> Resistor_SMD:R_0805_2012Metric_Pad1.20x1.40mm_HandSolder
- R13: renamed from R21; footprint (none) -> Resistor_SMD:R_0805_2012Metric_Pad1.20x1.40mm_HandSolder
- R4: renamed from R23; footprint (none) -> Resistor_SMD:R_0805_2012Metric_Pad1.20x1.40mm_HandSolder
- R5: renamed from R17; footprint (none) -> Resistor_SMD:R_0805_2012Metric_Pad1.20x1.40mm_HandSolder
- R9: renamed from R24; value ~ -> 10k; footprint (none) -> Resistor_SMD:R_0805_2012Metric_Pad1.20x1.40mm_HandSolder
- renumbered J15 to J11, J22 to J16, J8 to J17, J9 to J18, J10 to J19, J16 to J2, J11 to J20, J12 to J3, J13 to J4, J17 to J6, J14 to J7, J18 to J8, J19 to J9, U2 to U1
Connections:
- net +3V3: now also D4.2 (A), C10.2, J10.1 (Pin_1), U2.7 (VOUT), U2.8 (VOUT)
- net +5V: now also C12.1, C13.1
- net PACK-: no longer J5.1 (Pin_1)
- net PGND_BAT: now also C5.2, C1.2, C12.2, C13.2, C3.2, C6.2, R2.2, R6.1, R8.2, U2.10 (PGND), U2.11 (PGND), U2.15 (PGND), U2.3 (PGND)
- net SGND: now also J5.1 (Pin_1), C10.1, J12.1 (Pin_1), J13.1 (Pin_1), J14.1 (Pin_1), J15.1 (Pin_1), R3.2, R6.2, R8.1, U2.12 (AGND); no longer C5.2
- net VBAT: now also C1.1, C3.1, C6.1, U2.1 (VIN), U2.14 (VIN), U2.2 (EN)
- net at R10.1, R9.2: now also U2.9 (FB)
- new net: R7.1, U2.13 (V5V)
- new net: R7.2, U2.6 (PGOOD)
- new net GND: R2.1, R3.1
Other:
- note removed: "Buck 외부 회로 부품 선정"
- moved on the sheet: C2, C4, C5, C7, C8, C9, D1, D2, D3, D4, J11, J16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
